Commit message: add urdf with joints

File: urdf/ieg55_with_joints.urdf.xacro (robot description, xacro)
@@ -22,4 +22,21 @@
             </visual>
         </link>
+        <joint name="${prefix}jaw_position" type="prismatic">
+            <parent link="${prefix}base"/>
+            <child link="${prefix}finger_right"/>
+            <origin rpy="0.0 0.0 ${pi}" xyz="0.0 -0.0115 0.045"/>
+            <axis xyz="1 0 0"/>
+            <limit effort="100.0" lower="0.0" upper="0.01" velocity="100.0"/>
+        </joint>
+        <link name="${prefix}finger_right"/>
+        <joint name="${prefix}jaw_position_mimic" type="prismatic">
+            <parent link="${prefix}base"/>
+            <child link="${prefix}finger_left"/>
+            <origin rpy="0.0 0.0 0.0" xyz="0.0 0.0115 0.045"/>
+            <axis xyz="1 0 0"/>
+            <limit effort="100.0" lower="0.0" upper="0.01" velocity="100.0"/>
+            <mimic joint="${prefix}jaw_position" multiplier="1"/>
+        </joint>
+        <link name="${prefix}finger_left"/>
         <joint name="${prefix}center" type="fixed">
             <parent link="${parent}"/>
